File: Hardware/Loud-Detector.kicad_sch (KiCad schematic)
At the start: 27 parts, among them J1 TP4056, J2 ON_OFF, J3 VIN+, J4 VIN-, J5 VOUT+, J6 VOUT-, J7 KY-037, Q1 BC557, Q2 BC547, U1 ATtiny85-20P, U2 MT3608_Module

Commit message: Adding schematics, PCB layout and base firmware
Parts:
- removed BZ1: Buzzer, Buzzer_Beeper:Buzzer_TDK_PS1240P02BT_D12.2mm_H6.5mm, symbol Device:Buzzer
- added J8: BUZZER, Connector_JST:JST_EH_B2B-EH-A_1x02_P2.50mm_Vertical, symbol Connector_Generic:Conn_01x02
- J7: footprint Connector_JST:JST_EH_B4B-EH-A_1x04_P2.50mm_Vertical -> Connector_JST:JST_EH_B3B-EH-A_1x03_P2.50mm_Vertical; symbol Connector_Generic:Conn_01x04 -> Connector_Generic:Conn_01x03
- R3, R4: footprint Resistor_THT:R_Axial_DIN0207_L6.3mm_D2.5mm_P2.54mm_Vertical -> Resistor_THT:R_Axial_DIN0207_L6.3mm_D2.5mm_P7.62mm_Horizontal
- U1: value ATtiny85-20P -> ATtiny85
Connections:
- net +5V: now also RV1.3, RV2.1; no longer RV1.1, RV2.3
- net GND: now also J7.2 (Pin_2), RV1.1; no longer J7.3 (Pin_3), RV1.3
- net LED2: now also U1.7 (PB2); no longer U1.2 (XTAL1/PB3)
- net MIC_OUT: now also J7.3 (Pin_3), U1.3 (XTAL2/PB4); no longer J7.4 (Pin_4), U1.7 (PB2)
- net THRESHOLD: now also U1.2 (XTAL1/PB3); no longer U1.3 (XTAL2/PB4)
- net VBAT+: now also J1.2 (Pin_2); no longer J1.1 (Pin_1)
- net VIN-: now also J1.1 (Pin_1); no longer J1.2 (Pin_2)
- net at C3.2, Q1.1 (C): now also J7.1 (Pin_1); no longer J7.2 (Pin_2)
- net at Q2.1 (C): now also J8.2 (Pin_2)
- net at RV2.2: now also J8.1 (Pin_1)
Other:
- moved on the sheet: H1, H2, RV2
